File: v2/rev-/xfer-sw_interface.sch (KiCad schematic (older format))
At the start: 51 parts, among them J1 CONTROL, J2 XFER_SW, J3 28VDC_IN, Q1 IRLML9301, Q2 IRLML9301, Q3 IRLML9301, Q4 IRLML9301, Q5 MMBTA06LT1G, Q6 MMBTA06LT1G, U1 ILD207T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

Commit message: version 2 of xfer switch interface design.  This commit sent to osh park 20220119
Parts:
- added TP1: +5V, TestPoint:TestPoint_Pad_D1.5mm, symbol Connector:TestPoint
- added TP10, TP4: ~P1, TestPoint:TestPoint_Pad_2.0x2.0mm, symbol Connector:TestPoint
- added TP11, TP5: ~P2, TestPoint:TestPoint_Pad_2.0x2.0mm, symbol Connector:TestPoint
- added TP12, TP6: ~INH, TestPoint:TestPoint_Pad_2.0x2.0mm, symbol Connector:TestPoint
- added TP13, TP7: ~I1_CTL, TestPoint:TestPoint_Pad_2.0x2.0mm, symbol Connector:TestPoint
- added TP14, TP8: ~I2_CTL, TestPoint:TestPoint_Pad_2.0x2.0mm, symbol Connector:TestPoint
- added TP15, TP9: GND, TestPoint:TestPoint_Pad_2.0x2.0mm, symbol Connector:TestPoint
- added TP2: +28V, TestPoint:TestPoint_Pad_D1.5mm, symbol Connector:TestPoint
- added TP3: GND, TestPoint:TestPoint_Pad_D1.5mm, symbol Connector:TestPoint
Connections:
- net +28V: now also TP2.1
- net +5V: now also TP1.1
- net C1+: now also TP10.1
- net C2+: now also TP12.1
- net GND: now also TP11.1, TP14.1, TP3.1, TP9.1
- net I1: now also TP13.1
- net I2: now also TP15.1
- net ~I1_CTL: now also TP7.1
- net ~I2_CTL: now also TP8.1
- net ~INH: now also TP6.1
- net ~P1: now also TP4.1
- net ~P2: now also TP5.1
Other:
- note added: "C1+ & C2+ to Positive \nSide of Relay Coils.\nRelay Coil Common (C-)\nis grounded."
- note added: "I1 & I2 to Indicator Switch. \nCommon Connector of Indicator Switch is grounded\nSignal is LOW to indicate position"
- note added: "Indicator Selector:\n- Default Position: LOW via optoisolator\n- Alternate Position:\n - Cut Solder Jumper Trace\n - Select direct path to Indicator on XFER switch\n - Transfer Switch Indicator Common is grounded so\n LOW signal still indicates switch position\n - Do not need LEDs, ILD207T, or 5Vreg: Do Not Populate"
- note added: "Pull Low to INHIBIT\nchange of position"
- note added: "Pulse Low to set \nPosition to P1"
- note added: "Pulse Low to set \nPosition to P2"
- note removed: "Indicator Selector:\n- Default Position: LOW via optoisolator\n- Alternate Position:\n - Cut Solder Jumper Trace\n - Select direct path to Indicator on XFER switch\n - Do not need LEDs, ILD207T, or 5Vreg: Do Not Populate"
- moved on the sheet: C5, C6, D5, D6, H1, H2, H3, H4, J3, JP1, JP2, Q3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
